Commit message: correcion inercias

File: taller_RM/src/mi_robot_diferencial/urdf/mi_robot.urdf.xacro (robot description, xacro)
@@ -14,5 +14,5 @@
     <inertial>
       <mass value="6.0"/>
-      <inertia ixx="0.01" ixy="0.0" ixz="0.0" iyy="0.01" iyz="0.0" izz="0.01"/>
+      <inertia ixx="0.03125" ixy="0.0" ixz="0.0" iyy="0.25625" iyz="0.0" izz="0.26500"/>
     </inertial>
   </link>
@@ -28,5 +28,5 @@
       <inertial>
         <mass value="1.0"/>
-        <inertia ixx="0.0005" ixy="0.0" ixz="0.0" iyy="0.0005" iyz="0.0" izz="0.0005"/>
+        <inertia ixx="0.00583" ixy="0.0" ixz="0.0" iyy="0.0058333" iyz="0.0" izz="0.01125"/>
       </inertial>
     </link>
